File: Application Board/Application.sch (EAGLE design)
At the start: 54 parts, among them Q1 DMP2012SN-7, T1 FDN340P, T2 AP1117_LIN_REG, U1 LM3409HV'LM3409HV'

Commit message: Changed some names, added vias
Parts:
- C_F, C_IN1, C_IN2: device eagle-ltspice:CC0603 -> resistor:C-USC0603
- C_OFF: device eagle-ltspice:CC0402 -> resistor:C-USC0603
- U1: value LM3409HV'LM3409HV' -> LM3409HV
- U2: value MAX3051MAX3051 -> MAX3051
- U3: value AP1117_LIN_REG -> U3
- renumbered ASV to Y1, T2 to U3, U$5 to U2
Changed lines of the file:
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@@
 <part name="C9" library="rcl" deviceset="C-US" device="C0603" value="0.1uF"/>
 <part name="C10" library="rcl" deviceset="C-US" device="C0603" value="1uF"/>
-<part name="ASV" library="DiscreteComponents" deviceset="ASF*" device="" value="8.000MHZ"/>
+<part name="Y1" library="DiscreteComponents" deviceset="ASF*" device="" value="8.000MHZ"/>
 <part name="C11" library="rcl" deviceset="C-US" device="C0603" value="0.1uF"/>
 <part name="GND2" library="supply1" deviceset="GND" device=""/>
@@
 <part name="R6" library="rcl" deviceset="R-US_" device="R0603" value="82"/>
 <part name="GND7" library="supply1" deviceset="GND" device=""/>
-<part name="U$5" library="MAX3051 Library" deviceset="MAX3051" device="MAX3051"/>
+<part name="U2" library="MAX3051 Library" deviceset="MAX3051" device="MAX3051" value="MAX3051"/>
 <part name="GND8" library="SparkFun-Aesthetics" deviceset="GND" device=""/>
 <part name="GND9" library="SparkFun-Aesthetics" deviceset="GND" device=""/>
@@
 <part name="R13" library="rcl" deviceset="R-US_" device="R0603" value="120"/>
 <part name="R14" library="rcl" deviceset="R-US_" device="R0603" value="100K"/>
-<part name="T2" library="PowerComponents" deviceset="AP1117_LIN_REG" device=""/>
+<part name="U3" library="PowerComponents" deviceset="AP1117_LIN_REG" device="" value="U3"/>
 <part name="C12" library="rcl" deviceset="C-US" device="C0603" value="0.22uF"/>
 <part name="C14" library="rcl" deviceset="C-US" device="C0603" value="0.22uF"/>
@@
 <part name="D6" library="DiscreteComponents" deviceset="SL12-E3/61T" device=""/>
 <part name="Q1" library="DiscreteComponents" deviceset="DMP2012SN-7" device=""/>
-<part name="C_F" library="eagle-ltspice" deviceset="C" device="C0603" value="1.0uF"/>
-<part name="C_IN2" library="eagle-ltspice" deviceset="C" device="C0603" value="2.2uF"/>
-<part name="C_IN1" library="eagle-ltspice" deviceset="C" device="C0603" value="2.2uF"/>
-<part name="C_OFF" library="eagle-ltspice" deviceset="C" device="C0402" value="470pF"/>
+<part name="C_F" library="resistor" deviceset="C-US" device="C0603" value="1.0uF"/>
+<part name="C_IN2" library="resistor" deviceset="C-US" device="C0603" value="2.2uF"/>
+<part name="C_IN1" library="resistor" deviceset="C-US" device="C0603" value="2.2uF"/>
+<part name="C_OFF" library="resistor" deviceset="C-US" device="C0603" value="470pF"/>
 <part name="GND12" library="supply1" deviceset="GND" device=""/>
 <part name="GND13" library="supply1" deviceset="GND" device=""/>
@@
 <part name="GND16" library="supply1" deviceset="GND" device=""/>
 <part name="GND17" library="supply1" deviceset="GND" device=""/>
-<part name="U1" library="2015_LED_Driver" deviceset="LM3409HV" device="'LM3409HV'"/>
+<part name="U1" library="2015_LED_Driver" deviceset="LM3409HV" device="'LM3409HV'" value="LM3409HV"/>
 <part name="FRAME3" library="frames" deviceset="FRAME_A_L" device=""/>
 <part name="U$2" library="Connectors" deviceset="HSCPART" device=""/>
@@
 <instance part="C9" gate="G$1" x="58.42" y="109.22"/>
 <instance part="C10" gate="G$1" x="45.72" y="109.22"/>
-<instance part="ASV" gate="G$1" x="185.42" y="165.1"/>
+<instance part="Y1" gate="G$1" x="185.42" y="165.1"/>
 <instance part="C11" gate="G$1" x="203.2" y="45.72"/>
 <instance part="GND2" gate="1" x="167.64" y="154.94"/>
@@
 <instance part="R6" gate="G$1" x="447.04" y="48.26" rot="R180"/>
 <instance part="GND7" gate="1" x="474.98" y="38.1"/>
-<instance part="U$5" gate="G$1" x="459.74" y="137.16"/>
+<instance part="U2" gate="G$1" x="459.74" y="137.16"/>
 <instance part="GND8" gate="1" x="444.5" y="114.3"/>
 <instance part="GND9" gate="1" x="487.68" y="124.46"/>
@@
 <instance part="R13" gate="G$1" x="482.6" y="139.7" rot="R270"/>
 <instance part="R14" gate="G$1" x="480.06" y="129.54"/>
-<instance part="T2" gate="G$1" x="353.06" y="139.7"/>
+<instance part="U3" gate="G$1" x="353.06" y="139.7"/>
 <instance part="C12" gate="G$1" x="340.36" y="137.16"/>
 <instance part="C14" gate="G$1" x="373.38" y="137.16"/>
@@
 <instance part="R_PD" gate="G$1" x="30.48" y="-133.35"/>
 <instance part="L1" gate="G$1" x="96.52" y="-151.13" rot="R90"/>
-<instance part="D6" gate="G$1" x="86.36" y="-156.21" rot="R90"/>
-<instance part="Q1" gate="G$1" x="78.74" y="-151.13" rot="R270"/>
+<instance part="D6" gate="G$1" x="86.36" y="-156.21" smashed="yes" rot="R90">
+<attribute name="NAME" x="84.455" y="-158.496" size="1.778" layer="95" rot="R90"/>
+<attribute name="VALUE" x="88.011" y="-153.924" size="0.8128" layer="96" rot="R270"/>
+</instance>
+<instance part="Q1" gate="G$1" x="78.74" y="-151.13" smashed="yes" rot="R270">
+<attribute name="VALUE" x="77.216" y="-148.082" size="0.8128" layer="96"/>
+<attribute name="NAME" x="78.994" y="-146.304" size="1.778" layer="95"/>
+</instance>
 <instance part="C_F" gate="G$1" x="78.74" y="-128.27" rot="R270"/>
 <instance part="C_IN2" gate="G$1" x="96.52" y="-128.27"/>
@@
 <pinref part="C7" gate="G$1" pin="2"/>
 <wire x1="167.64" y1="157.48" x2="167.64" y2="160.02" width="0.1524" layer="91"/>
-<pinref part="ASV" gate="G$1" pin="GND"/>
+<pinref part="Y1" gate="G$1" pin="GND"/>
 <wire x1="172.72" y1="160.02" x2="167.64" y2="160.02" width="0.1524" layer="91"/>
 <junction x="167.64" y="160.02"/>
@@
 </segment>
 <segment>
-<pinref part="U$5" gate="G$1" pin="GND"/>
+<pinref part="U2" gate="G$1" pin="GND"/>
 <wire x1="447.04" y1="129.54" x2="444.5" y2="129.54" width="0.1524" layer="91"/>
 <wire x1="444.5" y1="129.54" x2="444.5" y2="116.84" width="0.1524" layer="91"/>
@@
 <wire x1="353.06" y1="129.54" x2="373.38" y2="129.54" width="0.1524" layer="91"/>
 <wire x1="373.38" y1="129.54" x2="373.38" y2="132.08" width="0.1524" layer="91"/>
-<pinref part="T2" gate="G$1" pin="GND"/>
+<pinref part="U3" gate="G$1" pin="GND"/>
 <wire x1="353.06" y1="134.62" x2="353.06" y2="129.54" width="0.1524" layer="91"/>
 <junction x="353.06" y="129.54"/>
@@
 <net name="OSCIN" class="0">
 <segment>
-<pinref part="ASV" gate="G$1" pin="FO"/>
+<pinref part="Y1" gate="G$1" pin="FO"/>
 <wire x1="198.12" y1="165.1" x2="205.74" y2="165.1" width="0.1524" layer="91"/>
 <pinref part="U$1" gate="G$7" pin="PH0_OSCIN"/>
@@
 </segment>
 <segment>
-<pinref part="ASV" gate="G$1" pin="VCC"/>
+<pinref part="Y1" gate="G$1" pin="VCC"/>
 <wire x1="172.72" y1="170.18" x2="167.64" y2="170.18" width="0.1524" layer="91"/>
 <wire x1="167.64" y1="170.18" x2="167.64" y2="175.26" width="0.1524" layer="91"/>
@@
 </segment>
 <segment>
-<pinref part="U$5" gate="G$1" pin="VCC"/>
+<pinref part="U2" gate="G$1" pin="VCC"/>
 <wire x1="447.04" y1="144.78" x2="444.5" y2="144.78" width="0.1524" layer="91"/>
 <pinref part="+3V6" gate="G$1" pin="+3V3"/>
@@
 <segment>
 <pinref part="C14" gate="G$1" pin="1"/>
-<pinref part="T2" gate="G$1" pin="VOUT"/>
+<pinref part="U3" gate="G$1" pin="VOUT"/>
 <wire x1="373.38" y1="139.7" x2="373.38" y2="142.24" width="0.1524" layer="91"/>
 <wire x1="373.38" y1="142.24" x2="365.76" y2="142.24" width="0.1524" layer="91"/>
@@
 <wire x1="330.2" y1="142.24" x2="340.36" y2="142.24" width="0.1524" layer="91"/>
 <junction x="330.2" y="142.24"/>
-<pinref part="T2" gate="G$1" pin="VIN"/>
+<pinref part="U3" gate="G$1" pin="VIN"/>
 <pinref part="C12" gate="G$1" pin="1"/>
 <wire x1="340.36" y1="142.24" x2="342.9" y2="142.24" width="0.1524" layer="91"/>
@@
 <net name="CANL" class="0">
 <segment>
-<pinref part="U$5" gate="G$1" pin="CANL"/>
+<pinref part="U2" gate="G$1" pin="CANL"/>
 <wire x1="472.44" y1="134.62" x2="482.6" y2="134.62" width="0.1524" layer="91"/>
 <pinref part="R13" gate="G$1" pin="2"/>
@@
 <wire x1="482.6" y1="144.78" x2="477.52" y2="144.78" width="0.1524" layer="91"/>
 <wire x1="477.52" y1="144.78" x2="477.52" y2="139.7" width="0.1524" layer="91"/>
-<pinref part="U$5" gate="G$1" pin="CANH"/>
+<pinref part="U2" gate="G$1" pin="CANH"/>
 <wire x1="477.52" y1="139.7" x2="472.44" y2="139.7" width="0.1524" layer="91"/>
 <pinref part="R13" gate="G$1" pin="1"/>
@@
 <net name="N$63" class="0">
 <segment>
-<pinref part="U$5" gate="G$1" pin="RS"/>
+<pinref part="U2" gate="G$1" pin="RS"/>
 <pinref part="R14" gate="G$1" pin="1"/>
 <wire x1="474.98" y1="129.54" x2="472.44" y2="129.54" width="0.1524" layer="91"/>
@@
 </segment>
 <segment>
-<pinref part="U$5" gate="G$1" pin="RXD"/>
+<pinref part="U2" gate="G$1" pin="RXD"/>
 <wire x1="447.04" y1="134.62" x2="441.96" y2="134.62" width="0.1524" layer="91"/>
 <label x="434.34" y="134.62" size="1.778" layer="95"/>
@@
 </segment>
 <segment>
-<pinref part="U$5" gate="G$1" pin="TXD"/>
+<pinref part="U2" gate="G$1" pin="TXD"/>
 <wire x1="447.04" y1="139.7" x2="441.96" y2="139.7" width="0.1524" layer="91"/>
 <label x="434.34" y="139.7" size="1.778" layer="95"/>
